File: Nano-Tek.kicad_pcb (KiCad board)
At the start: 4 copper layers, 55 x 42 mm, 47 parts, among them CN1 POWER_IN, CN2 USB, CN3 Floppy 34, J1 Sound, J2 USB_Prog, J3 OLED+SER, J4 Encoder, Q1 MMBT3904, U1 STM32F105RBT6, U2 74LCX07, U3 AP2112K-3.3, X1 8MHz

Commit message: Changed project name as Nano-Tek
Parts:
- CN1: footprint gotek_compact:171826-4 -> Nano-Tek:171826-4
- CN2: footprint gotek_compact:USB-C-SMD_TYPE-C16PIN -> Nano-Tek:USB-C-SMD_TYPE-C16PIN
- LOGO1: footprint gotek_compact:NanoTek_Logo_Stacked_10mm -> Nano-Tek:NanoTek_Logo_Stacked_10mm
- LOGO2: footprint gotek_compact:NanoTek_Logo_Horizontal_Tagline -> Nano-Tek:NanoTek_Logo_Horizontal_Tagline
Changed lines of the file:
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@@
 	)
 	(paper "User" 132 110)
+	(title_block
+		(title "Vinny, Mesarim, Screemo, Kavanoz, Wrangler, Ordyne")
+		(date "2026-07-23")
+		(rev "1.0")
+		(company "Schematics derived from OpenFlops design by SukkoPera")
+	)
 	(layers
 		(0 "F.Cu" signal)
@@
 		(property ki_fp_filters "C_*")
 		(sheetname "/")
-		(sheetfile "gotek_compact.kicad_sch")
+		(sheetfile "Nano-Tek.kicad_sch")
 		(units
 			(unit
@@
 		(property ki_fp_filters "C_*")
 		(sheetname "/")
-		(sheetfile "gotek_compact.kicad_sch")
+		(sheetfile "Nano-Tek.kicad_sch")
 		(units
 			(unit
@@
 		(property ki_fp_filters "R_*")
 		(sheetname "/")
-		(sheetfile "gotek_compact.kicad_sch")
+		(sheetfile "Nano-Tek.kicad_sch")
 		(units
 			(unit
@@
 		(property ki_fp_filters "R_*")
 		(sheetname "/")
-		(sheetfile "gotek_compact.kicad_sch")
+		(sheetfile "Nano-Tek.kicad_sch")
 		(units
 			(unit
@@
 		(property ki_fp_filters "C_*")
 		(sheetname "/")
-		(sheetfile "gotek_compact.kicad_sch")
+		(sheetfile "Nano-Tek.kicad_sch")
 		(units
 			(unit
@@
 		(property ki_fp_filters "C_*")
 		(sheetname "/")
-		(sheetfile "gotek_compact.kicad_sch")
+		(sheetfile "Nano-Tek.kicad_sch")
 		(units
 			(unit
@@
 		(property ki_fp_filters "R_*")
 		(sheetname "/")
-		(sheetfile "gotek_compact.kicad_sch")
+		(sheetfile "Nano-Tek.kicad_sch")
 		(units
 			(unit
@@
 		(property ki_fp_filters "C_*")
 		(sheetname "/")
-		(sheetfile "gotek_compact.kicad_sch")
+		(sheetfile "Nano-Tek.kicad_sch")
 		(units
 			(unit
@@
 		(property ki_fp_filters "SOT?23?5*")
 		(sheetname "/")
-		(sheetfile "gotek_compact.kicad_sch")
+		(sheetfile "Nano-Tek.kicad_sch")
 		(units
 			(unit
@@
 		(property ki_fp_filters "C_*")
 		(sheetname "/")
-		(sheetfile "gotek_compact.kicad_sch")
+		(sheetfile "Nano-Tek.kicad_sch")
 		(units
 			(unit
@@
 		(property ki_fp_filters "R_*")
 		(sheetname "/")
-		(sheetfile "gotek_compact.kicad_sch")
+		(sheetfile "Nano-Tek.kicad_sch")
 		(units
 			(unit
@@
 		(property ki_fp_filters "R_*")
 		(sheetname "/")
-		(sheetfile "gotek_compact.kicad_sch")
+		(sheetfile "Nano-Tek.kicad_sch")
 		(units
 			(unit
@@
 		(property ki_fp_filters "R_*")
 		(sheetname "/")
-		(sheetfile "gotek_compact.kicad_sch")
+		(sheetfile "Nano-Tek.kicad_sch")
 		(units
 			(unit
@@
 		(property ki_fp_filters "C_*")
 		(sheetname "/")
-		(sheetfile "gotek_compact.kicad_sch")
+		(sheetfile "Nano-Tek.kicad_sch")
 		(units
 			(unit
@@
 		(property ki_fp_filters "R_*")
 		(sheetname "/")
-		(sheetfile "gotek_compact.kicad_sch")
+		(sheetfile "Nano-Tek.kicad_sch")
 		(units
 			(unit
@@
 		(property ki_fp_filters "C_*")
 		(sheetname "/")
-		(sheetfile "gotek_compact.kicad_sch")
+		(sheetfile "Nano-Tek.kicad_sch")
 		(units
 			(unit
@@
 		(property ki_fp_filters "MountingHole*Pad*")
 		(sheetname "/")
-		(sheetfile "gotek_compact.kicad_sch")
+		(sheetfile "Nano-Tek.kicad_sch")
 		(units
 			(unit
@@
 		(embedded_fonts no)
 	)
-	(footprint "gotek_compact:171826-4"
+	(footprint "Nano-Tek:171826-4"
 		(layer "F.Cu")
 		(at 86 19.95 -90)
@@
 		)
 		(sheetname "/")
-		(sheetfile "gotek_compact.kicad_sch")
+		(sheetfile "Nano-Tek.kicad_sch")
 		(units
 			(unit
@@
 		(property ki_fp_filters "C_*")
 		(sheetname "/")
-		(sheetfile "gotek_compact.kicad_sch")
+		(sheetfile "Nano-Tek.kicad_sch")
 		(units
 			(unit
@@
 		(property ki_fp_filters "R_*")
 		(sheetname "/")
-		(sheetfile "gotek_compact.kicad_sch")
+		(sheetfile "Nano-Tek.kicad_sch")
 		(units
 			(unit
@@
 		(property ki_fp_filters "R_*")
 		(sheetname "/")
-		(sheetfile "gotek_compact.kicad_sch")
+		(sheetfile "Nano-Tek.kicad_sch")
 		(units
 			(unit
@@
 		(property ki_fp_filters "MountingHole*Pad*")
 		(sheetname "/")
-		(sheetfile "gotek_compact.kicad_sch")
+		(sheetfile "Nano-Tek.kicad_sch")
 		(units
 			(unit
@@
 		(property ki_fp_filters "SOIC*3.9x8.7mm*P1.27mm* TSSOP*4.4x5mm*P0.65mm* DIP*W7.62mm*")
 		(sheetname "/")
-		(sheetfile "gotek_compact.kicad_sch")
+		(sheetfile "Nano-Tek.kicad_sch")
 		(units
 			(unit
@@
 		(property ki_fp_filters "R_*")
 		(sheetname "/")
-		(sheetfile "gotek_compact.kicad_sch")
+		(sheetfile "Nano-Tek.kicad_sch")
 		(units
 			(unit
@@
 		(property ki_fp_filters "Connector*:*_1x??_*")
 		(sheetname "/")
-		(sheetfile "gotek_compact.kicad_sch")
+		(sheetfile "Nano-Tek.kicad_sch")
 		(units
 			(unit
@@
 		)
 	)
-	(footprint "gotek_compact:NanoTek_Logo_Stacked_10mm"
+	(footprint "Nano-Tek:NanoTek_Logo_Stacked_10mm"
 		(layer "F.Cu")
 		(at 56 27.65)
@@
 		(property ki_fp_filters "R_*")
 		(sheetname "/")
-		(sheetfile "gotek_compact.kicad_sch")
+		(sheetfile "Nano-Tek.kicad_sch")
 		(units
 			(unit
@@
 		(property ki_fp_filters "C_*")
 		(sheetname "/")
-		(sheetfile "gotek_compact.kicad_sch")
+		(sheetfile "Nano-Tek.kicad_sch")
 		(units
 			(unit
@@
 		(property ki_fp_filters "Connector*:*_2x??_*")
 		(sheetname "/")
-		(sheetfile "gotek_compact.kicad_sch")
+		(sheetfile "Nano-Tek.kicad_sch")
 		(units
 			(unit
@@
 		(property ki_fp_filters "R_*")
 		(sheetname "/")
-		(sheetfile "gotek_compact.kicad_sch")
+		(sheetfile "Nano-Tek.kicad_sch")
 		(units
 			(unit
@@
 		(property ki_fp_filters "R_*")
 		(sheetname "/")
-		(sheetfile "gotek_compact.kicad_sch")
+		(sheetfile "Nano-Tek.kicad_sch")
 		(units
 			(unit
@@
 		(property ki_fp_filters "D*SOD?323*")
 		(sheetname "/")
-		(sheetfile "gotek_compact.kicad_sch")
+		(sheetfile "Nano-Tek.kicad_sch")
 		(units
 			(unit
@@
 		(property ki_fp_filters "Connector*:*_2x??_*")
 		(sheetname "/")
-		(sheetfile "gotek_compact.kicad_sch")
+		(sheetfile "Nano-Tek.kicad_sch")
 		(units
 			(unit
@@
 		(property ki_fp_filters "C_*")
 		(sheetname "/")
-		(sheetfile "gotek_compact.kicad_sch")
+		(sheetfile "Nano-Tek.kicad_sch")
 		(units
 			(unit
@@
 		(property ki_fp_filters "MountingHole*Pad*")
 		(sheetname "/")
-		(sheetfile "gotek_compact.kicad_sch")
+		(sheetfile "Nano-Tek.kicad_sch")
 		(units
 			(unit
@@
 		(property ki_fp_filters "LQFP*10x10mm*P0.5mm*")
 		(sheetname "/")
-		(sheetfile "gotek_compact.kicad_sch")
+		(sheetfile "Nano-Tek.kicad_sch")
 		(units
 			(unit
@@
 		(property ki_fp_filters "Crystal*")
 		(sheetname "/")
-		(sheetfile "gotek_compact.kicad_sch")
+		(sheetfile "Nano-Tek.kicad_sch")
 		(units
 			(unit
@@
 		)
 	)
-	(footprint "gotek_compact:USB-C-SMD_TYPE-C16PIN"
+	(footprint "Nano-Tek:USB-C-SMD_TYPE-C16PIN"
 		(layer "F.Cu")
 		(at 45.095 35.6 -90)
@@
 		)
 		(sheetname "/")
-		(sheetfile "gotek_compact.kicad_sch")
+		(sheetfile "Nano-Tek.kicad_sch")
 		(units
 			(unit
@@
 		(property ki_fp_filters "C_*")
 		(sheetname "/")
-		(sheetfile "gotek_compact.kicad_sch")
+		(sheetfile "Nano-Tek.kicad_sch")
 		(units
 			(unit
@@
 		(property ki_fp_filters "SOT?23*")
 		(sheetname "/")
-		(sheetfile "gotek_compact.kicad_sch")
+		(sheetfile "Nano-Tek.kicad_sch")
 		(units
 			(unit
@@
 		(property ki_fp_filters "Connector*:*_1x??_*")
 		(sheetname "/")
-		(sheetfile "gotek_compact.kicad_sch")
+		(sheetfile "Nano-Tek.kicad_sch")
 		(units
 			(unit
@@
 		(property ki_fp_filters "R_*")
 		(sheetname "/")
-		(sheetfile "gotek_compact.kicad_sch")
+		(sheetfile "Nano-Tek.kicad_sch")
 		(units
 			(unit
@@
 		(property ki_fp_filters "Connector*:*_1x??_*")
 		(sheetname "/")
-		(sheetfile "gotek_compact.kicad_sch")
+		(sheetfile "Nano-Tek.kicad_sch")
 		(units
 			(unit
@@
 		(property ki_fp_filters "C_*")
 		(sheetname "/")
-		(sheetfile "gotek_compact.kicad_sch")
+		(sheetfile "Nano-Tek.kicad_sch")
 		(units
 			(unit
@@
 		(property ki_fp_filters "MountingHole*Pad*")
 		(sheetname "/")
-		(sheetfile "gotek_compact.kicad_sch")
+		(sheetfile "Nano-Tek.kicad_sch")
 		(units
 			(unit
@@
 		(property ki_fp_filters "R_*")
 		(sheetname "/")
-		(sheetfile "gotek_compact.kicad_sch")
+		(sheetfile "Nano-Tek.kicad_sch")
 		(units
 			(unit
@@
 		)
 	)
-	(footprint "gotek_compact:NanoTek_Logo_Horizontal_Tagline"
+	(footprint "Nano-Tek:NanoTek_Logo_Horizontal_Tagline"
 		(layer "B.Cu")
 		(at 67.45 36.3 180)
